File: kicad/scheme.kicad_sch (KiCad schematic)
At the start: 46 parts, among them J1 reset, Q1 G1, SW1 SW_PUSH_6mm_H4.3mm, SW2 SW_PUSH_6mm_H4.3mm, SW3 SW_PUSH_6mm_H4.3mm, SW4 btn-start, SW5 SW_PUSH_6mm_H4.3mm, U1 COM-09032-103-530, U2 ESP-12E-no_pins, U3 PCA9306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

Commit message: kicad-updates
Parts:
- removed ICM-conn1: AUX-ICM-no!, Connector_PinHeader_2.54mm:PinHeader_1x04_P2.54mm_Vertical, symbol Connector:Conn_01x04_Pin
- added J2: Conn_01x04, Connector_PinSocket_2.54mm:PinSocket_1x04_P2.54mm_Vertical, symbol Connector_Generic:Conn_01x04
- added J3: poweron, Connector_PinHeader_2.54mm:PinHeader_2x01_P2.54mm_Vertical, symbol Connector:Conn_01x02_Pin
- added R16: R-100, Resistor_SMD:R_0805_2012Metric, symbol models:R-10k
- added R17: 4k7, Resistor_SMD:R_0805_2012Metric_Pad1.20x1.40mm_HandSolder, symbol Device:R_Small
- added R18: 1k, Resistor_SMD:R_0805_2012Metric_Pad1.20x1.40mm_HandSolder, symbol Device:R_Small
Connections:
- net +3.3V: now also R16.2
- net +4.2V: now also J2.1 (Pin_1), J3.1 (Pin_1); no longer TP4056-module1.3 (out+)
- net GND: now also J2.2 (Pin_2), R18.2; no longer SW4.1 (C)
- net SCL: now also J2.3 (Pin_3)
- net SDA: now also J2.4 (Pin_4)
- net bt+: now reaches BT1.+, TP4056-module1.5 (b+)
- net bt+: now also R17.1
- net at R6.1, U2.16 (GPIO15): now also SW4.1 (C)
- net at U2.2 (ADC): now also R17.2, R18.1; no longer SW4.2 (D)
- net aux-da: no longer names the net of U7.21 (AUX_DA)
- net aux_cl: no longer names the net of U7.7 (AUX_CL)
- new net: J3.2 (Pin_2), TP4056-module1.3 (out+)
- new net: R16.1, SW4.2 (D)
Other:
- note added: "ICM-version"
- moved on the sheet: C1, C10, C2, C3, C4, C5, C7, R12, R2, R3, R6, SW4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

Commit message: changes in scheme
Parts:
- removed J3: poweron, Connector_PinHeader_2.54mm:PinHeader_2x01_P2.54mm_Vertical, symbol Connector:Conn_01x02_Pin
- added S1: SLW-883935-2A-D, module-custom-for-esp8266:SW_SLW-883935-2A-D, symbol models:SLW-883935-2A-D
- C1, C10, C2, C3, C4, C5, C8, C9: footprint Capacitor_SMD:C_0805_2012Metric -> Resistor_SMD:R_0805_2012Metric_Pad1.20x1.40mm_HandSolder
- C7: footprint Capacitor_THT:CP_Radial_D10.0mm_P3.50mm -> Resistor_SMD:R_0805_2012Metric_Pad1.20x1.40mm_HandSolder
- R11, R12, R13, R14, R15, R16, R4, R5, R6, R7, R8: footprint Resistor_SMD:R_0805_2012Metric -> Resistor_SMD:R_0805_2012Metric_Pad1.20x1.40mm_HandSolder
Connections:
- net +4.2V: now also S1.3
- net GND: now also R6.1; no longer R6.2
- net at TP4056-module1.3 (out+): now also S1.2
- net at SW4.1 (C), U2.16 (GPIO15): now also R6.2; no longer R6.1
Other:
- moved on the sheet: C1, C3, R6, U4

Commit message: added Readme
Parts:
- S1: footprint module-custom-for-esp8266:SW_SLW-883935-2A-D -> module-custom-for-esp8266:SW_OS102011MS2QN1_slideSwitch; symbol models:SLW-883935-2A-D -> models:OS102011MS2QN1_SlideSwitch; MP SLW-883935-2A-D -> OS102011MS2QN1
Connections:
- net +3.3V: now also J2.1 (Pin_1)
- net +4.2V: now also S1.2; no longer J2.1 (Pin_1), S1.3
- net at TP4056-module1.3 (out+): now also S1.1; no longer S1.2

Commit message: udpate in scheme
Parts:
- removed TP4056-module1: ~, module-custom-for-esp8266:TP4056-Module, symbol models:TP4056-module
- added TP1: SDO, TestPoint:TestPoint_Pad_1.0x1.0mm, symbol Connector:TestPoint
- added TP2: SDA_1.8, TestPoint:TestPoint_Pad_1.0x1.0mm, symbol Connector:TestPoint
- added TP3: SCL_1.8, TestPoint:TestPoint_Pad_1.0x1.0mm, symbol Connector:TestPoint
- added TP4: CS, TestPoint:TestPoint_Pad_1.0x1.0mm, symbol Connector:TestPoint
- added TP4056-module1: ~, module-custom-for-esp8266:TP4056-short, symbol models:TP4056-module_short
- added TP5: 1.8V, TestPoint:TestPoint_Pad_1.0x1.0mm, symbol Connector:TestPoint
- C7: value C_Electrolitic_3.3V -> 0.1uF
- SW4: value btn-start -> btnB
Connections:
- net +1.8V: now also TP5.1
- net +5C: now also S1.3, TP4056-module1.1 (dc+)
- net GND: now also BT1.-, TP4056-module1.2 (dc-), TP4056-module1.4 (b-)
- net SCL_1.8: now also TP3.1
- net SDA_1.8: now also TP2.1
- net bt+: now also S1.1, TP4056-module1.3 (b+)
- net btnA: now also SW2.2 (D); no longer SW3.2 (D)
- net btnX: now also SW3.2 (D); no longer SW1.2 (D)
- net btnY: now also SW1.2 (D); no longer SW2.2 (D)
- net at R15.2, U7.22 (~{CS}): now also TP4.1
- net at R14.1, U7.9 (SDO/AD0): now also TP1.1
- net btnB renamed btn-trigger
Other:
- moved on the sheet: BT1, C1, C3, S1, SW1, SW2, SW3, U4

Commit message: update
Parts:
- added J3: AIN2-3, Connector_PinHeader_2.54mm:PinHeader_2x01_P2.54mm_Vertical, symbol Connector:Conn_01x02_Pin
Connections:
- net GND: no longer BT1.-
- net at U5.6 (AIN2): now also J3.1 (Pin_1)
- net at U5.7 (AIN3): now also J3.2 (Pin_2)
